Commit message: switch x,y coords/ Fix the thumb unnatural angles

File: openteach/robot/assets/robot.urdf (robot description, URDF)
Before this commit: robot onshape, 17 links, 16 joints
Joints:
- joint 14: limit lower=-1.20 upper=1.90 effort=0.95 velocity=8.48 -> lower=-1.2 upper=1.90 effort=0.95 velocity=8.48
